File: source/pcb/_restore_backup_2026-08-22T16-16-09-483/tesseract.kicad_pcb (KiCad board)
At the start: 2 copper layers, 83 parts, among them J1 USB_C_Receptacle_USB2.0_14P, J2 AudioJack3_SwitchTR, J3 Conn_01x12, J4 Conn_01x02, J5 Micro_SD_Card_Det1, SW1 SW_Push, SW2 SW_Push, SW3 SW_Push, SW4 SW_Push, SW5 SW_Push, SW6 SW_Push, U1 PCM5102A, U2 IP5306, U3 RP2354A, U4 XC6206PxxxMR, U5 PAM8403D, Y1 Crystal_GND24

Commit message: Assigned footprints to symbols
Parts:
- removed J5: Micro_SD_Card_Det1, Connector_Card:microSD_HC_Hirose_DM3BT-DSF-PEJS
- removed R15, R16, R17, R18: 10K, Resistor_SMD:R_0402_1005Metric
- J2: footprint footprints:PJ31060 -> Connector_Audio:Jack_3.5mm_PJ31060-I_Horizontal
Connections:
- U3 pad 16: unconnected-(U3-GPIO12-Pad16) -> GP12
- U3 pad 17: SDCD -> GP13
- U3 pad 18: SDSCK -> GP14
- U3 pad 19: SDMOSI -> GP15
- U3 pad 27: SDMISO -> GP16
- U3 pad 28: SDCS -> GP17
- U3 pad 29: unconnected-(U3-GPIO18-Pad29) -> GP18
- U3 pad 31: unconnected-(U3-GPIO19-Pad31) -> GP19
- U3 pad 32: unconnected-(U3-GPIO20-Pad32) -> GP20
- U3 pad 33: unconnected-(U3-GPIO21-Pad33) -> GP21
- U3 pad 34: unconnected-(U3-GPIO22-Pad34) -> GP22
- U3 pad 53: +3V3 -> unconnected-(U3-USB_OTP_VDD-Pad53)
