File: source/pcb/_restore_backup_2026-08-22T16-16-09-483/tesseract.kicad_sch (KiCad schematic)
At the start: 83 parts, among them J1 USB_C_Receptacle_USB2.0_14P, J2 AudioJack3_SwitchTR, J3 Conn_01x12, J4 Conn_01x02, J5 Micro_SD_Card_Det1, SW1 SW_Push, SW2 SW_Push, SW3 SW_Push, SW4 SW_Push, SW5 SW_Push, SW6 SW_Push, U1 PCM5102A, U2 IP5306, U3 RP2354A, U4 XC6206PxxxMR, U5 PAM8403D, Y1 Crystal_GND24

Commit message: Assigned footprints to symbols
Parts:
- J2: footprint footprints:PJ31060 -> Connector_Audio:Jack_3.5mm_PJ31060-I_Horizontal
- SW3, SW4, SW5, SW6: footprint Button_Switch_THT:SW_PUSH_6mm -> Button_Switch_SMD:SW_Push_1P1T_NO_CK_PTS125Sx43PSMTR
Changed lines of the file:
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@@
 			)
 		)
-		(property "Footprint" "Button_Switch_THT:SW_PUSH_6mm"
+		(property "Footprint" "Button_Switch_SMD:SW_Push_1P1T_NO_CK_PTS125Sx43PSMTR"
 			(at 179.07 125.73 0)
 			(hide yes)
@@
 			)
 		)
-		(property "Footprint" "footprints:PJ31060"
+		(property "Footprint" "Connector_Audio:Jack_3.5mm_PJ31060-I_Horizontal"
 			(at 252.73 71.12 0)
 			(hide yes)
@@
 			)
 		)
-		(property "Footprint" "Button_Switch_THT:SW_PUSH_6mm"
+		(property "Footprint" "Button_Switch_SMD:SW_Push_1P1T_NO_CK_PTS125Sx43PSMTR"
 			(at 232.41 125.73 0)
 			(hide yes)
@@
 			)
 		)
-		(property "Footprint" "Button_Switch_THT:SW_PUSH_6mm"
+		(property "Footprint" "Button_Switch_SMD:SW_Push_1P1T_NO_CK_PTS125Sx43PSMTR"
 			(at 196.85 125.73 0)
 			(hide yes)
@@
 			)
 		)
-		(property "Footprint" "Button_Switch_THT:SW_PUSH_6mm"
+		(property "Footprint" "Button_Switch_SMD:SW_Push_1P1T_NO_CK_PTS125Sx43PSMTR"
 			(at 214.63 125.73 0)
 			(hide yes)
