File: source/pcb/tesseract.kicad_sch (KiCad schematic)
At the start: 83 parts, among them J1 USB_C_Receptacle_USB2.0_14P, J2 AudioJack3_SwitchTR, J3 Conn_01x12, J4 Conn_01x02, J5 Micro_SD_Card_Det1, SW1 SW_Push, SW2 SW_Push, SW3 SW_Push, SW4 SW_Push, SW5 SW_Push, SW6 SW_Push, U1 PCM5102A, U2 IP5306, U3 RP2354A, U4 XC6206PxxxMR, U5 PAM8403D, Y1 Crystal_GND24

Commit message: Created PCB layout
Parts:
- removed SW5, SW6: SW_Push, Button_Switch_THT:SW_PUSH_6mm, symbol Switch:SW_Push
- SW1, SW2: footprint footprints:button_342 -> Inductor_SMD:L_Taiyo-Yuden_NR-40xx
- SW3, SW4: footprint Button_Switch_THT:SW_PUSH_6mm -> footprints:button_342
Connections:
- net +3V3: now also C43.1, U3.46 (VREG_AVDD)
- net GND: now also C43.2
- net B3: no longer names the net of U3.14 (GPIO10)
- net B4: no longer names the net of U3.15 (GPIO11)
- net VREG_AVDD: no longer names the net of C3.1, R5.2
- net VREG_AVDD: no longer U3.46 (VREG_AVDD)
- no-connect marks 26 -> 28

Commit message: Finished PCB routing
Parts:
- added H1, H2, H3, H4: MountingHole, MountingHole:MountingHole_3.2mm_M3, symbol Mechanical:MountingHole
- added H5: MountingHole, footprints:display_hole, symbol Mechanical:MountingHole
- J5: footprint Connector_Card:microSD_HC_Hirose_DM3BT-DSF-PEJS -> footprints:TF-SMD_TF-CARD-H1.8
Connections:
- net GND: now also J5.SH (SHIELD)

Commit message: Added slide switch and created firmware
Parts:
- added SW5: SW_SPDT, common_footprints:SW-TH_MSK12D18G2, symbol Switch:SW_SPDT
- H5: footprint footprints:display_hole -> common_footprints:display_hole
- J2: footprint footprints:PJ31060 -> common_footprints:PJ31060
- J5: footprint footprints:TF-SMD_TF-CARD-H1.8 -> common_footprints:TF-SMD_TF-CARD-H1.8
- U2: footprint footprints:eSOP-8 -> common_footprints:eSOP-8
Connections:
- net +3V3: now also SW5.1 (A); no longer C24.1, U4.2 (VO)
- net SDCD: now also U3.15 (GPIO11); no longer U3.17 (GPIO13)
- net SDCS: now also U3.17 (GPIO13); no longer U3.28 (GPIO17)
- net SDMISO: now also U3.16 (GPIO12); no longer U3.27 (GPIO16)
- new net: C24.1, SW5.2 (B), U4.2 (VO)
- no-connect marks 28 -> 29

Commit message: Added BOM
Parts:
- J2: footprint common_footprints:PJ31060 -> common_footprints:AUDIO-SMD_PJ-242_1
Changed lines of the file:
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@@
 			)
 		)
-		(property "Footprint" "common_footprints:PJ31060"
+		(property "Footprint" "common_footprints:AUDIO-SMD_PJ-242_1"
 			(at 252.73 71.12 0)
 			(hide yes)
